File: OpenAmigaDriveSwitcher.sch (KiCad schematic (older format))
At the start: 6 parts, among them J1 SWITCH, J99 OSHW_LOGO, U1 74LS157, U8 EVEN_CIA_CHIP

Commit message: Ready for V1
Parts:
- added J2: SWITCH, OpenAmigaDriveSwitcher:SolderJumper3, symbol Conn_01x03
- J1: footprint OpenAmigaDriveSwitcher:LoosePads-3 -> OpenAmigaDriveSwitcher:Pin_Header_Straight_1x03-ModSilkS
Connections:
- wire segments 149 -> 155
Other:
- moved on the sheet: J1
Changed lines of the file:
@@
 Sheet 1 1
 Title "OpenAmigaDriveSwitcher"
-Date "2018-06-25"
-Rev "1git"
-Comp ""
+Date "2018-06-26"
+Rev "1"
+Comp "SukkoPera"
 Comment1 ""
 Comment2 ""
@@
 L GND #PWR01
 U 1 1 5B3157DD
-P 4325 7500
-F 0 "#PWR01" H 4325 7250 50  0001 C CNN
-F 1 "GND" H 4325 7350 50  0000 C CNN
-F 2 "" H 4325 7500 50  0001 C CNN
-F 3 "" H 4325 7500 50  0001 C CNN
-	1    4325 7500
+P 4450 7500
+F 0 "#PWR01" H 4450 7250 50  0001 C CNN
+F 1 "GND" H 4450 7350 50  0000 C CNN
+F 2 "" H 4450 7500 50  0001 C CNN
+F 3 "" H 4450 7500 50  0001 C CNN
+	1    4450 7500
 	1    0    0    -1
 $EndComp
@@
 	4100 4650 7025 4650
 Wire Wire Line
-	4125 7350 5025 7350
-Wire Wire Line
-	4325 7350 4325 7500
+	4000 7350 5025 7350
+Wire Wire Line
+	4450 7350 4450 7500
 Wire Wire Line
 	4325 2575 4325 2850
@@
 L Conn_01x03 J1
 U 1 1 5B317465
-P 3925 7250
-F 0 "J1" H 3925 7450 50  0000 C CNN
-F 1 "SWITCH" H 3925 7050 50  0000 C CNN
-F 2 "OpenAmigaDriveSwitcher:LoosePads-3" H 3925 7250 50  0001 C CNN
-F 3 "" H 3925 7250 50  0001 C CNN
-	1    3925 7250
+P 3800 7250
+F 0 "J1" H 3800 7450 50  0000 C CNN
+F 1 "SWITCH" H 3800 7050 50  0000 C CNN
+F 2 "OpenAmigaDriveSwitcher:Pin_Header_Straight_1x03-ModSilkS" H 3800 7250 50  0001 C CNN
+F 3 "" H 3800 7250 50  0001 C CNN
+	1    3800 7250
 	-1   0    0    1
 $EndComp
 Wire Wire Line
-	4125 7250 5025 7250
-Connection ~ 4325 7350
-Wire Wire Line
-	4125 7150 4325 7150
-Wire Wire Line
-	4325 7150 4325 6975
+	4000 7250 5025 7250
+Connection ~ 4450 7350
+Wire Wire Line
+	4000 7150 4450 7150
+Wire Wire Line
+	4450 7150 4450 6975
 $Comp
 L VCC #PWR04
 U 1 1 5B3177E7
-P 4325 6975
-F 0 "#PWR04" H 4325 6825 50  0001 C CNN
-F 1 "VCC" H 4325 7125 50  0000 C CNN
-F 2 "" H 4325 6975 50  0001 C CNN
-F 3 "" H 4325 6975 50  0001 C CNN
-	1    4325 6975
+P 4450 6975
+F 0 "#PWR04" H 4450 6825 50  0001 C CNN
+F 1 "VCC" H 4450 7125 50  0000 C CNN
+F 2 "" H 4450 6975 50  0001 C CNN
+F 3 "" H 4450 6975 50  0001 C CNN
+	1    4450 6975
 	1    0    0    -1
 $EndComp
@@
 	4650 6750 4650 7350
 Connection ~ 4650 7350
+$Comp
+L Conn_01x03 J2
+U 1 1 5B327943
+P 3800 6625
+F 0 "J2" H 3800 6825 50  0000 C CNN
+F 1 "SWITCH" H 3800 6425 50  0000 C CNN
+F 2 "OpenAmigaDriveSwitcher:SolderJumper3" H 3800 6625 50  0001 C CNN
+F 3 "" H 3800 6625 50  0001 C CNN
+	1    3800 6625
+	-1   0    0    1
+$EndComp
+Wire Wire Line
+	4000 6725 4075 6725
+Wire Wire Line
+	4075 6725 4075 7350
+Connection ~ 4075 7350
+Wire Wire Line
+	4000 6625 4175 6625
+Wire Wire Line
+	4175 6625 4175 7250
+Connection ~ 4175 7250
+Wire Wire Line
+	4000 6525 4275 6525
+Wire Wire Line
+	4275 6525 4275 7150
+Connection ~ 4275 7150
 $EndSCHEMATC

Commit message: V2: Reverse swap pin logic (i.e: swap drives when it is grounded) This will make the switcher more easily controllable by OpenAmigaMouseTrigger. Also migrate project to KiCad 5.
Parts:
- C1: symbol C -> OpenAmigaDriveSwitcher-rescue:C
- CONN1: symbol EVEN_CIA_SOCKET -> EVEN_CIA_SOCKET:EVEN_CIA_SOCKET
- J1, J2: symbol Conn_01x03 -> OpenAmigaDriveSwitcher-rescue:Conn_01x03
- J99: symbol Conn_01x01 -> OpenAmigaDriveSwitcher-rescue:Conn_01x01
- U1: symbol 74LS157 -> OpenAmigaDriveSwitcher-rescue:74LS157
- U8: symbol EVEN_CIA_CHIP -> EVEN_CIA_CHIP:EVEN_CIA_CHIP
Connections:
- wire segments 155 -> 167
Changed lines of the file:
@@
-EESchema Schematic File Version 2
-LIBS:power
-LIBS:device
-LIBS:switches
-LIBS:relays
-LIBS:motors
-LIBS:transistors
-LIBS:conn
-LIBS:linear
-LIBS:regul
-LIBS:74xx
-LIBS:cmos4000
-LIBS:adc-dac
-LIBS:memory
-LIBS:xilinx
-LIBS:microcontrollers
-LIBS:dsp
-LIBS:microchip
-LIBS:analog_switches
-LIBS:motorola
-LIBS:texas
-LIBS:intel
-LIBS:audio
-LIBS:interface
-LIBS:digital-audio
-LIBS:philips
-LIBS:display
-LIBS:cypress
-LIBS:siliconi
-LIBS:opto
-LIBS:atmel
-LIBS:contrib
-LIBS:valves
-LIBS:EVEN_CIA_CHIP
-LIBS:EVEN_CIA_SOCKET
+EESchema Schematic File Version 4
 LIBS:OpenAmigaDriveSwitcher-cache
-EELAYER 25 0
+EELAYER 26 0
 EELAYER END
 $Descr A4 11693 8268
@@
 Sheet 1 1
 Title "OpenAmigaDriveSwitcher"
-Date "2018-06-26"
-Rev "1"
+Date "2018-08-18"
+Rev "2"
 Comp "SukkoPera"
 Comment1 ""
@@
 $EndDescr
 $Comp
-L EVEN_CIA_CHIP U8
+L EVEN_CIA_CHIP:EVEN_CIA_CHIP U8
 U 1 1 5B3150AF
 P 3350 3800
@@
 $EndComp
 $Comp
-L EVEN_CIA_SOCKET CONN1
+L EVEN_CIA_SOCKET:EVEN_CIA_SOCKET CONN1
 U 1 1 5B3150E2
 P 7775 3800
@@
 $EndComp
 $Comp
-L 74LS157 U1
+L OpenAmigaDriveSwitcher-rescue:74LS157 U1
 U 1 1 5B315560
 P 5775 6800
@@
 NoConn ~ 6525 7050
 $Comp
-L GND #PWR01
+L power:GND #PWR01
 U 1 1 5B3157DD
 P 4450 7500
@@
 $EndComp
 $Comp
-L VCC #PWR02
+L power:VCC #PWR02
 U 1 1 5B3158BB
 P 4325 2575
@@
 $EndComp
 Wire Wire Line
-	4100 4750 7025 4750
-Wire Wire Line
-	4100 2850 7025 2850
+	4100 4750 4325 4750
+Wire Wire Line
+	4100 2850 4325 2850
 Wire Wire Line
 	4100 2950 7025 2950
@@
 	4100 4650 7025 4650
 Wire Wire Line
-	4000 7350 5025 7350
+	4000 7350 4075 7350
 Wire Wire Line
 	4450 7350 4450 7500
@@
 Connection ~ 4325 2850
 $Comp
-L GND #PWR03
+L power:GND #PWR03
 U 1 1 5B315A06
 P 4325 4925
@@
 	4100 3550 4750 3550
 Wire Wire Line
-	4750 3550 4750 6600
-Wire Wire Line
-	4750 6250 5025 6250
-Wire Wire Line
-	4750 6600 5025 6600
-Connection ~ 4750 6250
-Wire Wire Line
 	4100 3450 4650 3450
 Wire Wire Line
-	4650 3450 4650 6500
-Wire Wire Line
-	4650 6350 5025 6350
-Wire Wire Line
-	4650 6500 5025 6500
-Connection ~ 4650 6350
-Wire Wire Line
 	6525 6300 6700 6300
 Wire Wire Line
@@
 	1850 4250 2600 4250
 $Comp
-L Conn_01x03 J1
+L OpenAmigaDriveSwitcher-rescue:Conn_01x03 J1
 U 1 1 5B317465
 P 3800 7250
@@
 $EndComp
 Wire Wire Line
-	4000 7250 5025 7250
+	4000 7250 4175 7250
 Connection ~ 4450 7350
 Wire Wire Line
-	4000 7150 4450 7150
+	4000 7150 4275 7150
 Wire Wire Line
 	4450 7150 4450 6975
 $Comp
-L VCC #PWR04
+L power:VCC #PWR04
 U 1 1 5B3177E7
 P 4450 6975
@@
 $EndComp
 $Comp
-L C C1
+L OpenAmigaDriveSwitcher-rescue:C C1
 U 1 1 5B317A3C
 P 3175 6750
@@
 $EndComp
 $Comp
-L VCC #PWR05
+L power:VCC #PWR05
 U 1 1 5B317BA8
 P 3175 6475
@@
 $EndComp
 $Comp
-L GND #PWR06
+L power:GND #PWR06
 U 1 1 5B317BC2
 P 3175 7050
@@
 	3175 6600 3175 6475
 $Comp
-L Conn_01x01 J99
+L OpenAmigaDriveSwitcher-rescue:Conn_01x01 J99
 U 1 1 5B317D78
 P 11025 6250
@@
 Connection ~ 4650 7350
 $Comp
-L Conn_01x03 J2
+L OpenAmigaDriveSwitcher-rescue:Conn_01x03 J2
 U 1 1 5B327943
 P 3800 6625
@@
 	4275 6525 4275 7150
 Connection ~ 4275 7150
+Wire Wire Line
+	4325 2850 7025 2850
+Wire Wire Line
+	4325 4750 7025 4750
+Wire Wire Line
+	4450 7350 4650 7350
+Wire Wire Line
+	4950 7350 5025 7350
+Wire Wire Line
+	4850 7350 4950 7350
+Wire Wire Line
+	4750 7350 4850 7350
+Wire Wire Line
+	4650 7350 4750 7350
+Wire Wire Line
+	4075 7350 4450 7350
+Wire Wire Line
+	4175 7250 5025 7250
+Wire Wire Line
+	4275 7150 4450 7150
+Wire Wire Line
+	4650 6600 5025 6600
+Wire Wire Line
+	4750 6500 5025 6500
+Wire Wire Line
+	4650 3450 4650 6250
+Wire Wire Line
+	4750 3550 4750 6350
+Wire Wire Line
+	5025 6350 4750 6350
+Connection ~ 4750 6350
+Wire Wire Line
+	4750 6350 4750 6500
+Wire Wire Line
+	5025 6250 4650 6250
+Connection ~ 4650 6250
+Wire Wire Line
+	4650 6250 4650 6600
 $EndSCHEMATC
